Commit message: Changed axis

File: urdf/centaur2.xacro (robot description, xacro)
@@ -318,5 +318,5 @@
   <parent link="wheelShaft_1"/>
   <child link="AERO-FLEX_WHEEL_v1_1"/>
-  <axis xyz="1.0 0.0 -0.0"/>
+  <axis xyz="1.0 -0.0 0.0"/>
 </joint>
 <joint name="Rev23" type="continuous">

Commit message: Redid previous chnage

File: urdf/centaur2.xacro (robot description, xacro)
@@ -318,5 +318,5 @@
   <parent link="wheelShaft_1"/>
   <child link="AERO-FLEX_WHEEL_v1_1"/>
-  <axis xyz="1.0 -0.0 0.0"/>
+  <axis xyz="1.0 0.0 -0.0"/>
 </joint>
 <joint name="Rev23" type="continuous">
