Commit message: Update

File: urdf/sentry.xacro (robot description, xacro)
@@ -7,5 +7,5 @@
   <inertial>
     <origin rpy="0 0 0" xyz="-2.14622738325042e-06 -1.2948856978626193e-07 0.17005643721843872"/>
-    <mass value="7.486731783757874"/>
+    <mass value="0.1"/>
     <inertia ixx="0.551048" ixy="2e-06" ixz="-2e-06" iyy="0.349591" iyz="-0.0" izz="0.508154"/>
   </inertial>

Commit message: Update

File: urdf/sentry.xacro (robot description, xacro)
@@ -6,7 +6,7 @@
 <link name="base_link">
   <inertial>
-    <origin rpy="0 0 0" xyz="-2.14622738325042e-06 -1.2948856978626193e-07 0.17005643721843872"/>
-    <mass value="0.1"/>
-    <inertia ixx="0.551048" ixy="2e-06" ixz="-2e-06" iyy="0.349591" iyz="-0.0" izz="0.508154"/>
+    <origin rpy="0 0 0" xyz="-1.675313026909233e-06 -1.0107684249866667e-07 0.1400116338734353"/>
+    <mass value="3.298877191482148"/>
+    <inertia ixx="0.245613" ixy="1e-06" ixz="-0.0" iyy="0.14737" iyz="-0.0" izz="0.236442"/>
   </inertial>
   <visual>

Commit message: Float robot test

File: urdf/sentry.xacro (robot description, xacro)
@@ -6,7 +6,7 @@
 <link name="base_link">
   <inertial>
-    <origin rpy="0 0 0" xyz="-1.675313026909233e-06 -1.0107684249866667e-07 0.1400116338734353"/>
-    <mass value="3.298877191482148"/>
-    <inertia ixx="0.245613" ixy="1e-06" ixz="-0.0" iyy="0.14737" iyz="-0.0" izz="0.236442"/>
+    <origin rpy="0 0 0" xyz="-2.6855944968741624e-07 -1.6203026454315877e-08 0.1056505116603424"/>
+    <mass value="20.57887719148214"/>
+    <inertia ixx="0.411001" ixy="1e-06" ixz="0.0" iyy="0.312757" iyz="0.0" izz="0.351642"/>
   </inertial>
   <visual>
@@ -26,10 +26,10 @@
 <link name="right_wheel__1__1">
   <inertial>
-    <origin rpy="0 0 0" xyz="0.18575296055764245 -1.0523620236589737e-06 0.08050621246218834"/>
+    <origin rpy="0 0 0" xyz="0.18575296055764245 -1.0523620236589735e-06 0.18050621246218834"/>
     <mass value="0.5441760889032027"/>
     <inertia ixx="0.001218" ixy="0.0" ixz="-0.0" iyy="0.000635" iyz="-0.0" izz="0.000635"/>
   </inertial>
   <visual>
-    <origin rpy="0 0 0" xyz="-0.0 -0.0 0.009325"/>
+    <origin rpy="0 0 0" xyz="-0.0 0.0 0.009325"/>
     <geometry>
       <mesh filename="package://sentry_description/meshes/right_wheel__1__1.stl" scale="0.001 0.001 0.001"/>
@@ -38,5 +38,5 @@
   </visual>
   <collision>
-    <origin rpy="0 0 0" xyz="-0.0 -0.0 0.009325"/>
+    <origin rpy="0 0 0" xyz="-0.0 0.0 0.009325"/>
     <geometry>
       <mesh filename="package://sentry_description/meshes/right_wheel__1__1.stl" scale="0.001 0.001 0.001"/>
@@ -46,10 +46,10 @@
 <link name="left_wheel_1">
   <inertial>
-    <origin rpy="0 0 0" xyz="-0.18575295351621832 -9.94356549852574e-07 0.06185630713235224"/>
+    <origin rpy="0 0 0" xyz="-0.1857529535162183 -9.943565498525738e-07 0.16185630713235225"/>
     <mass value="0.5441781170129456"/>
     <inertia ixx="0.001218" ixy="-0.0" ixz="0.0" iyy="0.000635" iyz="-0.0" izz="0.000635"/>
   </inertial>
   <visual>
-    <origin rpy="0 0 0" xyz="0.0 0.0 -0.009325"/>
+    <origin rpy="0 0 0" xyz="-0.0 -0.0 -0.009325"/>
     <geometry>
       <mesh filename="package://sentry_description/meshes/left_wheel_1.stl" scale="0.001 0.001 0.001"/>
@@ -58,5 +58,5 @@
   </visual>
   <collision>
-    <origin rpy="0 0 0" xyz="0.0 0.0 -0.009325"/>
+    <origin rpy="0 0 0" xyz="-0.0 -0.0 -0.009325"/>
     <geometry>
       <mesh filename="package://sentry_description/meshes/left_wheel_1.stl" scale="0.001 0.001 0.001"/>

Commit message: Block and two wheels test

File: urdf/sentry.xacro (robot description, xacro)
@@ -6,7 +6,7 @@
 <link name="base_link">
   <inertial>
-    <origin rpy="0 0 0" xyz="-1.675313026909233e-06 -1.0107684249866663e-07 0.1400116338734353"/>
-    <mass value="3.298877191482148"/>
-    <inertia ixx="0.245613" ixy="1e-06" ixz="-0.0" iyy="0.14737" iyz="-0.0" izz="0.236442"/>
+    <origin rpy="0 0 0" xyz="0.0 0.0 0.20013598166728927"/>
+    <mass value="125.69767187998065"/>
+    <inertia ixx="2.096323" ixy="0.0" ixz="0.0" iyy="2.098602" iyz="0.0" izz="0.839613"/>
   </inertial>
   <visual>
@@ -26,10 +26,10 @@
 <link name="left_wheel_1">
   <inertial>
-    <origin rpy="0 0 0" xyz="-0.18575295351621837 -9.943565498527106e-07 0.06185630713235231"/>
+    <origin rpy="0 0 0" xyz="-0.19105823931257043 -9.94356549852711e-07 0.3655760224098007"/>
     <mass value="0.5441781170129456"/>
     <inertia ixx="0.001218" ixy="-0.0" ixz="0.0" iyy="0.000635" iyz="-0.0" izz="0.000635"/>
   </inertial>
   <visual>
-    <origin rpy="0 0 0" xyz="-0.0 -0.0 -0.009325"/>
+    <origin rpy="0 0 0" xyz="0.0 0.0 -0.009425"/>
     <geometry>
       <mesh filename="package://sentry_description/meshes/left_wheel_1.stl" scale="0.001 0.001 0.001"/>
@@ -38,5 +38,5 @@
   </visual>
   <collision>
-    <origin rpy="0 0 0" xyz="-0.0 -0.0 -0.009325"/>
+    <origin rpy="0 0 0" xyz="0.0 0.0 -0.009425"/>
     <geometry>
       <mesh filename="package://sentry_description/meshes/left_wheel_1.stl" scale="0.001 0.001 0.001"/>
@@ -44,35 +44,35 @@
   </collision>
 </link>
-<link name="right_wheel__1__1">
+<link name="right_wheel__2__1">
   <inertial>
-    <origin rpy="0 0 0" xyz="0.18575296055764245 -1.0523620236589735e-06 0.08050621246218817"/>
+    <origin rpy="0 0 0" xyz="0.19105824635399465 -1.0523620236591105e-06 0.38442592773963674"/>
     <mass value="0.5441760889032027"/>
     <inertia ixx="0.001218" ixy="0.0" ixz="-0.0" iyy="0.000635" iyz="-0.0" izz="0.000635"/>
   </inertial>
   <visual>
-    <origin rpy="0 0 0" xyz="-0.0 -0.0 0.009325"/>
+    <origin rpy="0 0 0" xyz="-0.0 0.0 0.009425"/>
     <geometry>
-      <mesh filename="package://sentry_description/meshes/right_wheel__1__1.stl" scale="0.001 0.001 0.001"/>
+      <mesh filename="package://sentry_description/meshes/right_wheel__2__1.stl" scale="0.001 0.001 0.001"/>
     </geometry>
     <material name="silver"/>
   </visual>
   <collision>
-    <origin rpy="0 0 0" xyz="-0.0 -0.0 0.009325"/>
+    <origin rpy="0 0 0" xyz="-0.0 0.0 0.009425"/>
     <geometry>
-      <mesh filename="package://sentry_description/meshes/right_wheel__1__1.stl" scale="0.001 0.001 0.001"/>
+      <mesh filename="package://sentry_description/meshes/right_wheel__2__1.stl" scale="0.001 0.001 0.001"/>
     </geometry>
   </collision>
 </link>
 <joint name="left_wheel_joint" type="continuous">
-  <origin rpy="0 0 0" xyz="0.0 0.0 0.009325"/>
+  <origin rpy="0 0 0" xyz="0.0 0.0 0.009425"/>
   <parent link="base_link"/>
   <child link="left_wheel_1"/>
-  <axis xyz="-1.0 -0.0 -0.0"/>
+  <axis xyz="-1.0 0.0 0.0"/>
 </joint>
 <joint name="right_wheel_joint" type="continuous">
-  <origin rpy="0 0 0" xyz="0.0 0.0 -0.009325"/>
+  <origin rpy="0 0 0" xyz="0.0 0.0 -0.009425"/>
   <parent link="base_link"/>
-  <child link="right_wheel__1__1"/>
-  <axis xyz="1.0 -0.0 -0.0"/>
+  <child link="right_wheel__2__1"/>
+  <axis xyz="1.0 0.0 0.0"/>
 </joint>
 </robot>

Commit message: Updated trans

File: urdf/sentry.xacro (robot description, xacro)
@@ -6,5 +6,5 @@
 <link name="base_link">
   <inertial>
-    <origin rpy="0 0 0" xyz="1.1129913184308585e-14 0.0005217136280458697 0.0728451162666737"/>
+    <origin rpy="0 0 0" xyz="0 0 0"/>
     <mass value="98.47956252925857"/>
     <inertia ixx="2.141143" ixy="-0.0" ixz="0.0" iyy="0.596002" iyz="0.003043" izz="2.571777"/>
@@ -26,10 +26,11 @@
 <link name="wheel_1">
   <inertial>
-    <origin rpy="0 0 0" xyz="-0.16605823931256913 -0.20000099435655025 0.0635760224098007"/>
+    <!--<origin rpy="0 0 0" xyz="-0.16605823931256913 -0.20000099435655025 0.0635760224098007"/>-->
+    <origin rpy="0 0 0" xyz="0.165575 0.20000099435655025 -0.109"/>
     <mass value="0.5441781170129456"/>
     <inertia ixx="0.001218" ixy="-0.0" ixz="0.0" iyy="0.000635" iyz="-0.0" izz="0.000635"/>
   </inertial>
   <visual>
-    <origin rpy="0 0 0" xyz="-0.0 -0.0 -0.009425"/>
+    <origin rpy="0 0 0" xyz="0.165575 0.20000099435655025 -0.109"/>
     <geometry>
       <mesh filename="package://sentry_description/meshes/wheel_1.stl" scale="0.001 0.001 0.001"/>
@@ -38,5 +39,5 @@
   </visual>
   <collision>
-    <origin rpy="0 0 0" xyz="-0.0 -0.0 -0.009425"/>
+    <origin rpy="0 0 0" xyz="0.165575 0.20000099435655025 -0.109"/>
     <geometry>
       <mesh filename="package://sentry_description/meshes/wheel_1.stl" scale="0.001 0.001 0.001"/>
@@ -46,10 +47,11 @@
 <link name="wheel_2">
   <inertial>
-    <origin rpy="0 0 0" xyz="0.16605823931257102 -0.20000099435655025 0.0635739775901992"/>
+    <!--<origin rpy="0 0 0" xyz="0.16605823931257102 -0.20000099435655025 0.0635739775901992"/>-->
+    <origin rpy="0 0 0" xyz="-0.165575 0.20000099435655025 -0.109"/>
     <mass value="0.5441781170129456"/>
     <inertia ixx="0.001218" ixy="0.0" ixz="0.0" iyy="0.000635" iyz="0.0" izz="0.000635"/>
   </inertial>
   <visual>
-    <origin rpy="0 0 0" xyz="-0.0 -0.0 -0.009425"/>
+    <origin rpy="0 0 0" xyz="-0.165575 0.20000099435655025 -0.109"/>
     <geometry>
       <mesh filename="package://sentry_description/meshes/wheel_2.stl" scale="0.001 0.001 0.001"/>
@@ -58,5 +60,5 @@
   </visual>
   <collision>
-    <origin rpy="0 0 0" xyz="-0.0 -0.0 -0.009425"/>
+    <origin rpy="0 0 0" xyz="-0.165575 0.20000099435655025 -0.109"/>
     <geometry>
       <mesh filename="package://sentry_description/meshes/wheel_2.stl" scale="0.001 0.001 0.001"/>
@@ -65,14 +67,14 @@
 </link>
 <joint name="left_wheel_joint" type="continuous">
-  <origin rpy="0 0 0" xyz="0.0 0.0 0.009425"/>
+  <origin rpy="0 0 0" xyz="-0.165575 -0.20000099435655025 1"/>
   <parent link="base_link"/>
   <child link="wheel_1"/>
-  <axis xyz="-1.0 0.0 -0.0"/>
+  <axis xyz="1.0 0.0 0.0"/>
 </joint>
 <joint name="right_wheel_joint" type="continuous">
-  <origin rpy="0 0 0" xyz="0.0 0.0 0.009425"/>
+  <origin rpy="0 0 0" xyz="0.165575 -0.20000099435655025 1"/>
   <parent link="base_link"/>
   <child link="wheel_2"/>
-  <axis xyz="1.0 -0.0 0.0"/>
+  <axis xyz="1.0 0.0 0.0"/>
 </joint>
 </robot>

Commit message: Updated transmission

File: urdf/sentry.xacro (robot description, xacro)
@@ -27,10 +27,10 @@
   <inertial>
     <!--<origin rpy="0 0 0" xyz="-0.16605823931256913 -0.20000099435655025 0.0635760224098007"/>-->
-    <origin rpy="0 0 0" xyz="0.165575 0.20000099435655025 -0.109"/>
+    <origin rpy="0 0 0" xyz="0 0 0"/>
     <mass value="0.5441781170129456"/>
     <inertia ixx="0.001218" ixy="-0.0" ixz="0.0" iyy="0.000635" iyz="-0.0" izz="0.000635"/>
   </inertial>
   <visual>
-    <origin rpy="0 0 0" xyz="0.165575 0.20000099435655025 -0.109"/>
+    <origin rpy="0 0 0" xyz="0 0 0"/>
     <geometry>
       <mesh filename="package://sentry_description/meshes/wheel_1.stl" scale="0.001 0.001 0.001"/>
@@ -39,5 +39,5 @@
   </visual>
   <collision>
-    <origin rpy="0 0 0" xyz="0.165575 0.20000099435655025 -0.109"/>
+    <origin rpy="0 0 0" xyz="0 0 0"/>
     <geometry>
       <mesh filename="package://sentry_description/meshes/wheel_1.stl" scale="0.001 0.001 0.001"/>
@@ -48,10 +48,10 @@
   <inertial>
     <!--<origin rpy="0 0 0" xyz="0.16605823931257102 -0.20000099435655025 0.0635739775901992"/>-->
-    <origin rpy="0 0 0" xyz="-0.165575 0.20000099435655025 -0.109"/>
+    <origin rpy="0 0 0" xyz="0 0 0"/>
     <mass value="0.5441781170129456"/>
     <inertia ixx="0.001218" ixy="0.0" ixz="0.0" iyy="0.000635" iyz="0.0" izz="0.000635"/>
   </inertial>
   <visual>
-    <origin rpy="0 0 0" xyz="-0.165575 0.20000099435655025 -0.109"/>
+    <origin rpy="0 0 0" xyz="0 0 0"/>
     <geometry>
       <mesh filename="package://sentry_description/meshes/wheel_2.stl" scale="0.001 0.001 0.001"/>
@@ -60,5 +60,5 @@
   </visual>
   <collision>
-    <origin rpy="0 0 0" xyz="-0.165575 0.20000099435655025 -0.109"/>
+    <origin rpy="0 0 0" xyz="0 0 0"/>
     <geometry>
       <mesh filename="package://sentry_description/meshes/wheel_2.stl" scale="0.001 0.001 0.001"/>
@@ -67,5 +67,5 @@
 </link>
 <joint name="left_wheel_joint" type="continuous">
-  <origin rpy="0 0 0" xyz="-0.165575 -0.20000099435655025 1"/>
+  <origin rpy="0 0 1.57" xyz="-0.165575 -0.20000099435655025 0.109"/>
   <parent link="base_link"/>
   <child link="wheel_1"/>
@@ -73,5 +73,5 @@
 </joint>
 <joint name="right_wheel_joint" type="continuous">
-  <origin rpy="0 0 0" xyz="0.165575 -0.20000099435655025 1"/>
+  <origin rpy="0 0 1.57" xyz="0.165575 -0.20000099435655025 .109"/>
   <parent link="base_link"/>
   <child link="wheel_2"/>
